Commit message: making changes

File: catkin_ws/src/test_build/src/urdf/sick.urdf.xacro (robot description, xacro)
@@ -9,5 +9,5 @@
   </material>
   <!-- LMS291 Lidar model -->
-  <link name="lms291">
+  <link name="laser">
     <inertial>
       <mass value="4.5" />
@@ -33,5 +33,5 @@
   </link>
   <!-- LMS291 Lidar Mount model -->
-  <link name="lms291_mount">
+  <link name="laser_mount">
     <inertial>
       <mass value="0.4" />
@@ -58,6 +58,6 @@
   <joint name="lms291_to_mount" type="fixed">
     <origin xyz="0 -0.093 0.078" rpy="0 0 ${PI/(-2)}" />
-    <parent link="lms291_mount"/>
-    <child link="lms291"/>
+    <parent link="laser_mount"/>
+    <child link="laser"/>
   </joint>
   <!-- Link for Mount to Jackal -->
@@ -65,41 +65,5 @@
     <origin xyz="-0.090 0 0" rpy="0 0 ${PI/2}" />
     <parent link="front_mount"/>
-    <child link="lms291_mount"/>
+    <child link="laser_mount"/>
   </joint>
-  <gazebo reference="lms291">
-    <material>Gazebo/Blue</material>
-    <turnGravityOff>true</turnGravityOff>
-    <sensor type="ray" name="laser">
-      <pose>0 0 5 0 0 0</pose>
-      <visualize>true</visualize>
-      <update_rate>40</update_rate>
-      <ray>
-        <scan>
-          <horizontal>
-            <samples>720</samples>
-            <resolution>1</resolution>
-            <min_angle>-1.570796</min_angle>
-            <max_angle>1.570796</max_angle>
-          </horizontal>
-        </scan>
-        <range>
-          <min>0.10</min>
-          <max>30.0</max>
-          <resolution>0.01</resolution>
-        </range>
-        <noise>
-          <type>gaussian</type>
-          <mean>0.0</mean>
-          <stddev>0.01</stddev>
-        </noise>
-      </ray>
-      <plugin name="laser_plug" filename="libgazebo_ros_laser.so">
-        <topicName>/scan</topicName>
-        <frameName>lms291</frameName>
-      </plugin>
-    </sensor>
-  </gazebo>
-  <gazebo reference="lms291_mount">
-    <material>Gazebo/Grey</material>
-  </gazebo>
 </robot>

Commit message: Still trying stuff on the urdf

File: catkin_ws/src/test_build/src/urdf/sick.urdf.xacro (robot description, xacro)
@@ -9,5 +9,5 @@
   </material>
   <!-- LMS291 Lidar model -->
-  <link name="laser">
+  <link name="lms291">
     <inertial>
       <mass value="4.5" />
@@ -21,5 +21,5 @@
       <origin xyz="0 0 0" rpy="0 0 ${PI/1}" />
       <geometry>
-        <box size="0.155 .156 .185"/>
+        <mesh filename="package://ee5900_jackal_description/meshes/lms291_asm.stl" scale="0.001 0.001 0.001" />
       </geometry>
       <material name="blue"/>
@@ -33,5 +33,5 @@
   </link>
   <!-- LMS291 Lidar Mount model -->
-  <link name="laser_mount">
+  <link name="lms291_mount">
     <inertial>
       <mass value="0.4" />
@@ -44,5 +44,5 @@
     <visual>
       <geometry>
-        <mesh filename="package://test_build/src/meshes/LidarMount.stl" scale="0.001 0.001 0.001"/>
+        <mesh filename="package://ee5900_jackal_description/meshes/LidarMount.stl" scale="0.001 0.001 0.001"/>
       </geometry>
       <material name="grey"/>
@@ -58,6 +58,6 @@
   <joint name="lms291_to_mount" type="fixed">
     <origin xyz="0 -0.093 0.078" rpy="0 0 ${PI/(-2)}" />
-    <parent link="laser_mount"/>
-    <child link="laser"/>
+    <parent link="lms291_mount"/>
+    <child link="lms291"/>
   </joint>
   <!-- Link for Mount to Jackal -->
@@ -65,5 +65,5 @@
     <origin xyz="-0.090 0 0" rpy="0 0 ${PI/2}" />
     <parent link="front_mount"/>
-    <child link="laser_mount"/>
+    <child link="lms291_mount"/>
   </joint>
 </robot>

Commit message: Still trying stuff on the urdf

File: catkin_ws/src/test_build/src/urdf/sick.urdf.xacro (robot description, xacro)
@@ -21,5 +21,5 @@
       <origin xyz="0 0 0" rpy="0 0 ${PI/1}" />
       <geometry>
-        <mesh filename="package://ee5900_jackal_description/meshes/lms291_asm.stl" scale="0.001 0.001 0.001" />
+        <box size="0.155 .156 .185"/>
       </geometry>
       <material name="blue"/>
@@ -44,5 +44,5 @@
     <visual>
       <geometry>
-        <mesh filename="package://ee5900_jackal_description/meshes/LidarMount.stl" scale="0.001 0.001 0.001"/>
+        <mesh filename="package://test_build/src/meshes/LidarMount-1.stl" scale="0.001 0.001 0.001"/>
       </geometry>
       <material name="grey"/>
